File: Hypersoniq.kicad_pcb (KiCad board)
At the start: 2 copper layers, 72.2 x 72.2 mm, 70 parts, among them J1 Conn_01x05_Socket, J2 Conn_01x03_Socket, J3 Conn_01x05_Socket, J4 Conn_01x03_Socket, J5 Conn_01x01_Pin, SW1 ~{LP}_HP, U1 TL072, U2 DG442xY, U3 SSI2140, U4 SSI2140

Commit message: First draft of schematic
Parts:
- removed FREQ_POT1, locked: 10k, Custom_Footprints:Alpha_9mm_Potentiometer_Aligned
- removed J5: Conn_01x01_Pin, Connector_PinHeader_2.54mm:PinHeader_1x01_P2.54mm_Vertical
- removed SW1: ~{LP}_HP, Custom_Footprints:SPDTSubMiniature
- added C19: 1nF, Capacitor_SMD:C_0603_1608Metric_Pad1.08x0.95mm_HandSolder, F.Cu at (117.5, 102.0)
- added C20: 100nF, Capacitor_SMD:C_0603_1608Metric_Pad1.08x0.95mm_HandSolder, F.Cu at (117.5, 104.6)
- added C21: 100nF, Capacitor_SMD:C_0603_1608Metric_Pad1.08x0.95mm_HandSolder, F.Cu at (117.5, 107.1)
- added C22: 10nF, Capacitor_SMD:C_0603_1608Metric_Pad1.08x0.95mm_HandSolder, F.Cu at (121.8, 89.5)
- added C23: 2.2nF, Capacitor_SMD:C_0603_1608Metric_Pad1.08x0.95mm_HandSolder, F.Cu at (140.9, 67.4)
- added C24: 2.2nF, Capacitor_SMD:C_0603_1608Metric_Pad1.08x0.95mm_HandSolder, F.Cu at (140.9, 69.9)
- added C25: 1nF, Capacitor_SMD:C_0603_1608Metric_Pad1.08x0.95mm_HandSolder, F.Cu at (140.9, 72.4)
- added C26: 1nF, Capacitor_SMD:C_0603_1608Metric_Pad1.08x0.95mm_HandSolder, F.Cu at (140.9, 75.0)
- added C27: 1nF, Capacitor_SMD:C_0603_1608Metric_Pad1.08x0.95mm_HandSolder, F.Cu at (140.9, 77.5)
- added C28: 1nF, Capacitor_SMD:C_0603_1608Metric_Pad1.08x0.95mm_HandSolder, F.Cu at (140.9, 80.0)
- added C29: 100nF, Capacitor_SMD:C_0603_1608Metric_Pad1.08x0.95mm_HandSolder, F.Cu at (140.9, 82.5)
- added C30: 100nF, Capacitor_SMD:C_0603_1608Metric_Pad1.08x0.95mm_HandSolder, F.Cu at (140.9, 85.0)
- added C31: 10nF, Capacitor_SMD:C_0603_1608Metric_Pad1.08x0.95mm_HandSolder, F.Cu at (145.2, 67.4)
- added C32: 2.2nF, Capacitor_SMD:C_0603_1608Metric_Pad1.08x0.95mm_HandSolder, F.Cu at (117.5, 67.4)
- added C33: 2.2nF, Capacitor_SMD:C_0603_1608Metric_Pad1.08x0.95mm_HandSolder, F.Cu at (117.5, 69.9)
- added C34: 1nF, Capacitor_SMD:C_0603_1608Metric_Pad1.08x0.95mm_HandSolder, F.Cu at (117.5, 72.4)
- added C35: 1nF, Capacitor_SMD:C_0603_1608Metric_Pad1.08x0.95mm_HandSolder, F.Cu at (117.5, 75.0)
- added C36: 1nF, Capacitor_SMD:C_0603_1608Metric_Pad1.08x0.95mm_HandSolder, F.Cu at (117.5, 77.5)
- added C37: 1nF, Capacitor_SMD:C_0603_1608Metric_Pad1.08x0.95mm_HandSolder, F.Cu at (117.5, 80.0)
- added C38: 100nF, Capacitor_SMD:C_0603_1608Metric_Pad1.08x0.95mm_HandSolder, F.Cu at (117.5, 82.5)
- added C39: 100nF, Capacitor_SMD:C_0603_1608Metric_Pad1.08x0.95mm_HandSolder, F.Cu at (117.5, 85.0)
- added C40: 10nF, Capacitor_SMD:C_0603_1608Metric_Pad1.08x0.95mm_HandSolder, F.Cu at (121.8, 67.4)
- added C41: 100nF, Capacitor_SMD:C_0603_1608Metric_Pad1.08x0.95mm_HandSolder, F.Cu at (117.5, 48.5)
- added C42: 100nF, Capacitor_SMD:C_0603_1608Metric_Pad1.08x0.95mm_HandSolder, F.Cu at (117.5, 51.0)
- added D1: 1N5819, Diode_SMD:D_SOD-123, F.Cu at (88.6, 55.4)
- added D2: 1N5819, Diode_SMD:D_SOD-123, F.Cu at (51.8, 55.4)
- added Q_POT1: 10k, Custom_Footprints:Alpha_9mm_Potentiometer_Aligned, F.Cu at (135.5, 48.5)
- added R40: 1k, Resistor_SMD:R_0603_1608Metric_Pad0.98x0.95mm_HandSolder, F.Cu at (149.6, 69.9)
- added R41: 56k, Resistor_SMD:R_0603_1608Metric_Pad0.98x0.95mm_HandSolder, F.Cu at (149.6, 72.4)
- added R42: 100k, Resistor_SMD:R_0603_1608Metric_Pad0.98x0.95mm_HandSolder, F.Cu at (149.6, 75.0)
- added R43: 100k, Resistor_SMD:R_0603_1608Metric_Pad0.98x0.95mm_HandSolder, F.Cu at (149.6, 77.5)
- added R44: 50k, Resistor_SMD:R_0603_1608Metric_Pad0.98x0.95mm_HandSolder, F.Cu at (149.6, 80.0)
- added R45: 150k, Resistor_SMD:R_0603_1608Metric_Pad0.98x0.95mm_HandSolder, F.Cu at (149.6, 82.5)
- added R46: 200, Resistor_SMD:R_0603_1608Metric_Pad0.98x0.95mm_HandSolder, F.Cu at (121.8, 69.9)
- added R47: 200, Resistor_SMD:R_0603_1608Metric_Pad0.98x0.95mm_HandSolder, F.Cu at (121.8, 72.4)
- added R48: 200, Resistor_SMD:R_0603_1608Metric_Pad0.98x0.95mm_HandSolder, F.Cu at (121.8, 75.0)
- added R49: 200, Resistor_SMD:R_0603_1608Metric_Pad0.98x0.95mm_HandSolder, F.Cu at (121.8, 77.5)
- added R50: 10k, Resistor_SMD:R_0603_1608Metric_Pad0.98x0.95mm_HandSolder, F.Cu at (121.8, 80.0)
- added R51: 10k, Resistor_SMD:R_0603_1608Metric_Pad0.98x0.95mm_HandSolder, F.Cu at (121.8, 82.5)
- added R52: 10k, Resistor_SMD:R_0603_1608Metric_Pad0.98x0.95mm_HandSolder, F.Cu at (121.8, 85.0)
- added R53: 10k, Resistor_SMD:R_0603_1608Metric_Pad0.98x0.95mm_HandSolder, F.Cu at (126.2, 67.4)
- added R54: 1k, Resistor_SMD:R_0603_1608Metric_Pad0.98x0.95mm_HandSolder, F.Cu at (126.2, 69.9)
- added R55: 56k, Resistor_SMD:R_0603_1608Metric_Pad0.98x0.95mm_HandSolder, F.Cu at (126.2, 72.4)
- added R56: 100k, Resistor_SMD:R_0603_1608Metric_Pad0.98x0.95mm_HandSolder, F.Cu at (126.2, 75.0)
- added R57: 100k, Resistor_SMD:R_0603_1608Metric_Pad0.98x0.95mm_HandSolder, F.Cu at (126.2, 77.5)
- added R58: 50k, Resistor_SMD:R_0603_1608Metric_Pad0.98x0.95mm_HandSolder, F.Cu at (126.2, 80.0)
- added R59: 150k, Resistor_SMD:R_0603_1608Metric_Pad0.98x0.95mm_HandSolder, F.Cu at (126.2, 82.5)
- added R60: 10k, Resistor_SMD:R_0603_1608Metric_Pad0.98x0.95mm_HandSolder, F.Cu at (70.2, 18.5)
- added R61: 10k, Resistor_SMD:R_0603_1608Metric_Pad0.98x0.95mm_HandSolder, F.Cu at (70.2, 21.0)
- added R62: 10k, Resistor_SMD:R_0603_1608Metric_Pad0.98x0.95mm_HandSolder, F.Cu at (70.2, 23.5)
- added R63: 10k, Resistor_SMD:R_0603_1608Metric_Pad0.98x0.95mm_HandSolder, F.Cu at (70.2, 26.0)
- added R64: 4.7k, Resistor_SMD:R_0603_1608Metric_Pad0.98x0.95mm_HandSolder, F.Cu at (74.5, 18.5)
- added R65: 1k, Resistor_SMD:R_0603_1608Metric_Pad0.98x0.95mm_HandSolder, F.Cu at (74.5, 21.0)
- added R66: 10k, Resistor_SMD:R_0603_1608Metric_Pad0.98x0.95mm_HandSolder, F.Cu at (74.5, 23.5)
- added R67: 10k, Resistor_SMD:R_0603_1608Metric_Pad0.98x0.95mm_HandSolder, F.Cu at (74.5, 26.0)
- added R68: 10k, Resistor_SMD:R_0603_1608Metric_Pad0.98x0.95mm_HandSolder, F.Cu at (78.9, 18.5)
- added R69: 10k, Resistor_SMD:R_0603_1608Metric_Pad0.98x0.95mm_HandSolder, F.Cu at (78.9, 21.0)
- added R70: 4.7k, Resistor_SMD:R_0603_1608Metric_Pad0.98x0.95mm_HandSolder, F.Cu at (78.9, 23.5)
- added R71: 1k, Resistor_SMD:R_0603_1608Metric_Pad0.98x0.95mm_HandSolder, F.Cu at (78.9, 26.0)
- added TP2: TestPoint, Custom_Footprints:1.3mm_Test_Point, F.Cu at (56.8, 62.5)
- added TP3: TestPoint, Custom_Footprints:1.3mm_Test_Point, F.Cu at (88.4, 148.0)
- added TP4: TestPoint, Custom_Footprints:1.3mm_Test_Point, F.Cu at (80.4, 62.6)
- added U5: SSI2140, Package_SO:SSOP-20_4.4x6.5mm_P0.65mm, F.Cu at (132.5, 70.2)
- added U6: TL072, Package_SO:SO-8_3.9x4.9mm_P1.27mm, F.Cu at (72.2, 30.5)
- added kibuzzard-63F9EC4B: G***, kibuzzard-63F9EC4B, F.Cu at (51.6, 119.1)
- added kibuzzard-63F9ECEE: G***, kibuzzard-63F9ECEE, F.Cu at (88.7, 119.1)
- added kibuzzard-63FCE890: G***, kibuzzard-63FCE890, F.Cu at (51.6, 110.9)
- added kibuzzard-63FCEF0D: G***, kibuzzard-63FCEF0D, F.Cu at (88.7, 110.7)
- added kibuzzard-640237A8: G***, kibuzzard-640237A8, F.Cu at (84.1, 60.8)
- added kibuzzard-640237DF: G***, kibuzzard-640237DF, F.Cu at (80.4, 60.8)
- added kibuzzard-640237DF: G***, kibuzzard-640237DF, F.Cu at (88.5, 146.2)
- added kibuzzard-640237FD: G***, kibuzzard-640237FD, F.Cu at (56.9, 60.7)
- C1: value 22pF -> 22uF; footprint Capacitor_SMD:C_0603_1608Metric_Pad1.08x0.95mm_HandSolder -> Capacitor_SMD:CP_Elec_4x5.8
- C11, C3, C4: value 1nF -> 100nF
- C13: value 100nF -> 10nF
- C14: value 10nF -> 2.2nF
- C15, C6: value 100nF -> 2.2nF
- C16, C17, C18, C7: value 100nF -> 1nF
- C2: value 1nF -> 22uF; footprint Capacitor_SMD:C_0603_1608Metric_Pad1.08x0.95mm_HandSolder -> Capacitor_SMD:CP_Elec_4x5.8
- C5: value 1nF -> 2.2nF
- J1, J3: value Conn_01x05_Socket -> Conn_01x10_Pin; footprint Connector_PinSocket_2.54mm:PinSocket_1x05_P2.54mm_Vertical -> Connector_PinHeader_2.54mm:PinHeader_1x10_P2.54mm_Vertical; moved to B.Cu
- J2: value Conn_01x03_Socket -> Conn_01x10_Pin; footprint Connector_PinSocket_2.54mm:PinSocket_1x03_P2.54mm_Vertical -> Connector_PinHeader_2.54mm:PinHeader_1x10_P2.54mm_Vertical; moved to B.Cu
- J4: value Conn_01x03_Socket -> Eurorack_10_pin_power; footprint Connector_PinSocket_2.54mm:PinSocket_1x03_P2.54mm_Vertical -> Custom_Footprints:Eurorack_10_pin_header
- R1: value R_{A}_90k -> 39k
- R10, R22, R23, R24, R8, R9: value 200 -> 10k
- R11: value 15k -> 10k
- R12: value 15k -> 1k
- R13: value 15k -> 56k
- R14, R15: value 15k -> 100k
- R16: value 15k -> 50k
- R17: value 15k -> 150k
- R18: value 15k -> 200
- R19: value 1k -> 200
- R2: value R_{B}_22.5k -> 8.2k
- R20: value 54.9 -> 200
- R26: value 10k -> 1k
- R27: value 10k -> 56k
- R28: value 10k -> 100k
- R29: value 1k -> 100k
- R3: value R_{C}_15k -> 3.9k
- R30: value 54.9 -> 50k
- R31: value 100k -> 150k
- R32: value 100k -> 200
- R33: value 50k -> 200
- R34, R35: value 36k -> 200
- R36, R37: value 22k -> 10k
- R38: value 150k -> 10k
- R39: value 1k -> 10k
- R4: value R_{D}_22.5k -> 200
- R5: value R_{E}_90k -> 200
- R6: value R_{F}_90k -> 200
- U1: value TL072 -> TL074; footprint Package_SO:SO-8_3.9x4.9mm_P1.27mm -> Package_SO:SOIC-14_3.9x8.7mm_P1.27mm
- U2: value DG442xY -> SSI2140; footprint Package_SO:SOIC-16_3.9x9.9mm_P1.27mm -> Package_SO:SSOP-20_4.4x6.5mm_P0.65mm
- moved C10 147.4 mm to (211.7, 52.7), turned to 0 degrees
- moved R11 138.1 mm to (211.7, 54.3)
- moved C11 137.4 mm to (205.5, 58.4)
- moved R7 137.3 mm to (211.7, 55.9), turned to 0 degrees
- moved R12 136.7 mm to (211.7, 59.1)
- moved C9 136.6 mm to (211.7, 47.9), turned to 0 degrees
- moved C12 132.6 mm to (205.4, 48.4), turned to 180 degrees
- moved C6 130.1 mm to (211.7, 57.5)
- moved R6 127.7 mm to (211.7, 49.5), turned to 0 degrees
- moved C13 125.8 mm to (194.9, 53.7), turned to 180 degrees
- moved U2 125.6 mm to (205.5, 53.5)
- moved R13 124.3 mm to (199.3, 57.5), turned to 180 degrees
- moved R8 124.3 mm to (199.3, 55.9), turned to 0 degrees
- moved R10 123.2 mm to (211.7, 51.1)
- moved C8 122.7 mm to (199.3, 49.5), turned to 0 degrees
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Connections:
- C1 pad 1: /MM_MIX -> +12V
- C1 pad 2: Net-(C1-Pad2) -> GND
- C10 pad 1: Net-(U4-OUT2) -> Net-(U2-OUT3)
- C10 pad 2: Net-(U4-CAP3) -> Net-(U2-CAP4)
- C11 pad 1: Net-(U4-OUT3) -> -12V
- C11 pad 2: Net-(U4-CAP4) -> GND
- C12 pad 1: -12V -> +12V
- C13 pad 1: +12V -> Net-(U1A--)
- C13 pad 2: GND -> /Filter_Voice1/FREQ_CONTROL
- C14 pad 1: Net-(U1B--) -> Net-(U3-OUT1)
- C14 pad 2: /FREQ_CONTROL -> /1POLE_OUT2
- C15 pad 1: +12V -> /4POLE_OUT2
- C15 pad 2: GND -> Net-(U3-OUT4)
- C16 pad 1: -12V -> /AUDIO_IN2
- C16 pad 2: GND -> Net-(U3-CAP1)
- C17 pad 1: -12V -> Net-(U3-OUT1)
- C17 pad 2: GND -> Net-(U3-CAP2)
- C18 pad 1: +12V -> Net-(U3-OUT2)
- C18 pad 2: GND -> Net-(U3-CAP3)
- C2 pad 2: Net-(U3-CAP1) -> -12V
- C3 pad 1: GND -> +12V
- C3 pad 2: Net-(U3-CAP2) -> GND
- C4 pad 1: GND -> -12V
- C4 pad 2: Net-(U3-CAP3) -> GND
- C5 pad 1: GND -> Net-(U2-OUT1)
- C5 pad 2: Net-(U3-CAP4) -> /1POLE_OUT1
- C6 pad 1: -12V -> /4POLE_OUT1
- C6 pad 2: GND -> Net-(U2-OUT4)
- C7 pad 1: +12V -> /AUDIO_IN1
- C7 pad 2: GND -> Net-(U2-CAP1)
- C8 pad 1: /INPUT -> Net-(U2-OUT1)
- C8 pad 2: Net-(U4-CAP1) -> Net-(U2-CAP2)
- C9 pad 1: Net-(U4-OUT1) -> Net-(U2-OUT2)
- C9 pad 2: Net-(U4-CAP2) -> Net-(U2-CAP3)
- J1 pad 1: /INPUT -> /FREQ_POT_VH
- J1 pad 2: /OUTPUT -> /4POLE_OUT2
- J1 pad 3: /FREQ_CV1 -> /4POLE_OUT4
- J1 pad 4: /FREQ_CV2 -> /FREQ_POT_VL
- J1 pad 5: /Q_CV -> /FREQ_POT
- J2 pad 2: -12V -> /4POLE_OUT1
- J2 pad 3: GND -> /4POLE_OUT3
- J3 pad 1: /INPUT -> /AUDIO_IN3
- J3 pad 2: /OUTPUT -> /FREQ_CV4
- J3 pad 3: /FREQ_CV1 -> /1POLE_OUT1
- J3 pad 4: /FREQ_CV2 -> GND
- J3 pad 5: /Q_CV -> /AUDIO_IN4
- J4 pad 1: +12V -> /-12V_IN
- J4 pad 2: -12V -> /-12V_IN
- R1 pad 1: Net-(R1-Pad1) -> /Q_POT
- R1 pad 2: /MM_MIX -> /Q_CONTROL
- R10 pad 1: Net-(U3-IN4) -> Net-(U2-OUT3)
- R10 pad 2: GND -> Net-(U2-IN3)
- R11 pad 1: /INPUT_FB -> Net-(U2-OUT4)
- R11 pad 2: /INPUT -> Net-(U2-IN4)
- R12 pad 1: Net-(U3-OUT1) -> Net-(U2-Q_VCA_IN+)
- R12 pad 2: /INPUT_FB -> GND
- R13 pad 1: Net-(U3-IN2) -> Net-(U2-EXPO_CTRL)
- R13 pad 2: Net-(U3-OUT1) -> /Filter_Voice1/FREQ_CONTROL
- R14 pad 1: Net-(U3-OUT2) -> Net-(U1A--)
- R14 pad 2: Net-(U3-IN2) -> /FREQ_CV1
- R15 pad 1: Net-(U3-IN3) -> Net-(U1A--)
- R15 pad 2: Net-(U3-OUT2) -> /FREQ_JACK
- R16 pad 1: Net-(U3-OUT3) -> Net-(U1A--)
- R16 pad 2: Net-(U3-IN3) -> /FREQ_POT
- R17 pad 1: Net-(U3-IN4) -> /Filter_Voice1/FREQ_CONTROL
- R17 pad 2: Net-(U3-OUT3) -> Net-(U1A--)
- R18 pad 1: Net-(U3-OUT4) -> /Filter_Voice2/Q_FEEDBACK
- R18 pad 2: Net-(U3-IN4) -> GND
- R19 pad 1: Net-(U3-Q_VCA_IN+) -> Net-(U3-IN2)
- R2 pad 1: Net-(R2-Pad1) -> +12V
- R2 pad 2: /MM_MIX -> /FREQ_POT_VH
- R20 pad 1: Net-(U3-EXPO_CTRL) -> Net-(U3-IN3)
- R20 pad 2: /FREQ_CONTROL -> GND
- R21 pad 1: Net-(U4-IN1) -> Net-(U3-IN4)
- R22 pad 1: Net-(U4-IN2) -> Net-(U3-OUT1)
- R22 pad 2: GND -> /Filter_Voice2/Q_FEEDBACK
- R23 pad 1: Net-(U4-IN3) -> Net-(U3-OUT2)
- R23 pad 2: GND -> Net-(U3-IN2)
- R24 pad 1: Net-(U4-IN4) -> Net-(U3-OUT3)
- R24 pad 2: GND -> Net-(U3-IN3)
- R25 pad 1: Net-(U4-OUT1) -> Net-(U3-OUT4)
- R25 pad 2: Net-(U4-IN1) -> Net-(U3-IN4)
- R26 pad 1: Net-(U4-OUT2) -> Net-(U3-Q_VCA_IN+)
- R26 pad 2: Net-(U4-IN2) -> GND
- R27 pad 1: Net-(U4-OUT3) -> Net-(U3-EXPO_CTRL)
- R27 pad 2: Net-(U4-IN3) -> /Filter_Voice2/FREQ_CONTROL
- R28 pad 1: /OUTPUT -> Net-(U1B--)
- R28 pad 2: Net-(U4-IN4) -> /FREQ_CV2
- R29 pad 1: Net-(U4-Q_VCA_IN+) -> Net-(U1B--)
- R29 pad 2: GND -> /FREQ_JACK
- R3 pad 1: Net-(R3-Pad1) -> /FREQ_POT_VL
- R3 pad 2: /MM_MIX -> -12V
- R30 pad 1: Net-(U4-EXPO_CTRL) -> Net-(U1B--)
- R30 pad 2: /FREQ_CONTROL -> /FREQ_POT
- R31 pad 1: Net-(U1B--) -> /Filter_Voice2/FREQ_CONTROL
- R31 pad 2: /FREQ_CV1 -> Net-(U1B--)
- R32 pad 1: Net-(U1B--) -> /Filter_Voice3/Q_FEEDBACK
- R32 pad 2: /FREQ_CV2 -> GND
- R33 pad 1: Net-(U1B--) -> Net-(U4-IN2)
- R33 pad 2: /FREQ_POT -> GND
- R34 pad 1: +12V -> Net-(U4-IN3)
- R34 pad 2: Net-(FREQ_POT1-Pad1) -> GND
- R35 pad 1: Net-(FREQ_POT1-Pad3) -> Net-(U4-IN4)
- R35 pad 2: -12V -> GND
- R36 pad 1: /Q_CV -> Net-(U4-OUT1)
- R36 pad 2: /Q_CONTROL -> /Filter_Voice3/Q_FEEDBACK
- R37 pad 1: Net-(Q_POT1-Pad2) -> Net-(U4-OUT2)
- R37 pad 2: /Q_CONTROL -> Net-(U4-IN2)
- R38 pad 1: /FREQ_CONTROL -> Net-(U4-OUT3)
- R38 pad 2: Net-(U1B--) -> Net-(U4-IN3)
- R39 pad 1: /OUTPUT -> Net-(U4-OUT4)
- R39 pad 2: Net-(C1-Pad2) -> Net-(U4-IN4)
- R4 pad 1: Net-(R4-Pad1) -> /Filter_Voice1/Q_FEEDBACK
- R4 pad 2: /MM_MIX -> GND
- R5 pad 1: Net-(U3-OUT4) -> Net-(U2-IN2)
- R5 pad 2: /MM_MIX -> GND
- R6 pad 1: Net-(C1-Pad2) -> Net-(U2-IN3)
- R6 pad 2: /MM_MIX -> GND
- R7 pad 1: /INPUT_FB -> Net-(U2-IN4)
- R8 pad 1: Net-(U3-IN2) -> Net-(U2-OUT1)
- R8 pad 2: GND -> /Filter_Voice1/Q_FEEDBACK
- R9 pad 1: Net-(U3-IN3) -> Net-(U2-OUT2)
- R9 pad 2: GND -> Net-(U2-IN2)
- TP1 pad 1: GND -> +12V
- U1 pad 1: Net-(C1-Pad2) -> /Filter_Voice1/FREQ_CONTROL
- U1 pad 2: /MM_MIX -> Net-(U1A--)
- U1 pad 4: -12V -> +12V
- U1 pad 7: /FREQ_CONTROL -> /Filter_Voice2/FREQ_CONTROL
- U1 pad 8: +12V -> /Filter_Voice3/FREQ_CONTROL
- U2 pad 1: /~{LP}_HP -> Net-(U2-OUT2)
- U2 pad 10: Net-(R3-Pad1) -> GND
- U2 pad 11: Net-(U3-OUT2) -> -12V
- U2 pad 12: unconnected-(U2E-NC-Pad12) -> /Q_CONTROL
- U2 pad 13: +12V -> Net-(U2-Q_VCA_IN+)
- U2 pad 14: Net-(U3-OUT3) -> Net-(U2-OUT4)
- U2 pad 15: Net-(R4-Pad1) -> Net-(U2-CAP4)
- U2 pad 16: /~{LP}_HP -> Net-(U2-IN4)
- U2 pad 2: Net-(R1-Pad1) -> Net-(U2-CAP2)
- U2 pad 3: /INPUT -> Net-(U2-IN2)
- U2 pad 4: -12V -> Net-(U2-OUT1)
- U2 pad 5: GND -> Net-(U2-CAP1)
- U2 pad 6: Net-(R2-Pad1) -> /Filter_Voice1/Q_FEEDBACK
- U2 pad 7: Net-(U3-OUT1) -> Net-(U2-EXPO_CTRL)
- U2 pad 8: /~{LP}_HP -> Net-(U2-EXPO_CTRL)
- U2 pad 9: /~{LP}_HP -> /Filter_Voice1/Q_FEEDBACK
- U3 pad 6: /INPUT_FB -> /Filter_Voice2/Q_FEEDBACK
- U3 pad 9: /INPUT_FB -> /Filter_Voice2/Q_FEEDBACK
- U4 pad 14: /OUTPUT -> Net-(U4-OUT4)
- U4 pad 6: Net-(U4-IN1) -> /Filter_Voice3/Q_FEEDBACK
- U4 pad 9: /INPUT -> /Filter_Voice3/Q_FEEDBACK
Routing:
- net +12V: track 233.0 -> 3.02 mm, vias 5 -> 0
- net -12V: track 182.6 -> 2.97 mm, vias 5 -> 0
- net /INPUT: track 130.0 -> 0.00 mm, vias 2 -> 0
- net /Q_CONTROL: track 104.0 -> 0.00 mm, vias 4 -> 0
- net /Q_CV: track 78.6 -> 0.00 mm
- net /MM_MIX: track 69.3 -> 0.00 mm
- net /~{LP}_HP: track 58.7 -> 0.00 mm, vias 2 -> 0
- net /OUTPUT: track 57.7 -> 0.00 mm, vias 2 -> 0
- net Net-(U3-OUT2): track 57.6 -> 0.00 mm
- net /FREQ_CONTROL: track 46.9 -> 0.00 mm, vias 2 -> 0
- net Net-(U4-OUT3): track 44.1 -> 0.00 mm
- net Net-(U4-IN4): track 34.1 -> 0.00 mm
- net Net-(U3-OUT1): track 29.8 -> 0.00 mm
- net Net-(U4-OUT2): track 27.8 -> 0.00 mm
- net Net-(U3-OUT3): track 27.6 -> 0.00 mm
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- added copper zone on In1.Cu, net GND
- added copper zone on In2.Cu, net GND
Other:
- board size 72.2 x 72.2 mm -> 40.4 x 100 mm
- copper layers 2 -> 4
- board text added: "J1"
- board text added: "J2"
- board text added: "J3"
- board text removed: "+12V"
- board text removed: "-12V"
- board text removed: "AUD IN"
- board text removed: "AUD OUT"
- board text removed: "CUTOFF"
- board text removed: "FREQ CV1"
- board text removed: "FREQ CV2"
- board text removed: "GND"
- board text removed: "HP"
- board text removed: "High Pass"
- board text removed: "LP"
- board text removed: "MultiMode"
- board text removed: "Q CV"
- board text removed: "RESONANCE"
- board text removed: "SSI2140 Multimode/High Pass Filter Test Board v1.0 2023 Mountjoy Modular"

Commit message: Revert "Revert "PCB Layout""
This reverts commit 17ea893c43406ccb0184a474adf0eed468bf1595.
Parts:
- removed Q_POT1: 10k, Custom_Footprints:Alpha_9mm_Potentiometer_Aligned
- removed kibuzzard-63F9EC4B: G***, kibuzzard-63F9EC4B
- removed kibuzzard-63F9ECEE: G***, kibuzzard-63F9ECEE
- removed kibuzzard-63FCE890: G***, kibuzzard-63FCE890
- removed kibuzzard-63FCEF0D: G***, kibuzzard-63FCEF0D
- moved R14 146.8 mm to (56.8, 105.2)
- moved R15 146.8 mm to (56.8, 106.8)
- moved R17 142.1 mm to (63.1, 105.2), turned to 180 degrees
- moved C13 142.1 mm to (63.1, 106.8), turned to 0 degrees
- moved R16 140.9 mm to (63.1, 108.4)
- moved C11 138.0 mm to (70.2, 85.6)
- moved C12 138.0 mm to (70.1, 75.6)
- moved U2 138.0 mm to (70.2, 80.6)
- moved R10 138.0 mm to (76.4, 78.2)
- moved R4 138.0 mm to (64.0, 86.2)
- moved C5 138.0 mm to (64.0, 75.0)
- moved C7 138.0 mm to (64.0, 81.4)
- moved C8 138.0 mm to (64.0, 76.6)
- moved R13 138.0 mm to (64.0, 84.6)
- moved R5 138.0 mm to (64.0, 79.8)
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Connections:
- C22 pad 1: Net-(U1B--) -> Net-(U1D--)
- C40 pad 1: Net-(U1D--) -> Net-(U1B--)
- J1 pad 1: /FREQ_POT_VH -> /FREQ_POT_VL
- J1 pad 10: /AUDIO_IN2 -> /FREQ_CV1
- J1 pad 3: /4POLE_OUT4 -> /4POLE_OUT3
- J1 pad 4: /FREQ_POT_VL -> /4POLE_OUT4
- J1 pad 5: /FREQ_POT -> /AUDIO_MIX_4POLE
- J1 pad 7: /FREQ_CV1 -> /1POLE_OUT1
- J1 pad 9: /AUDIO_MIX -> /AUDIO_IN1
- J2 pad 3: /4POLE_OUT3 -> /FREQ_POT_VH
- J2 pad 5: GND -> /AUDIO_MIX_1POLE
- J2 pad 8: /AUDIO_IN1 -> /AUDIO_IN2
- J3 pad 1: /AUDIO_IN3 -> /FREQ_CV3
- J3 pad 10: /FREQ_CV3 -> /FREQ_JACK
- J3 pad 2: /FREQ_CV4 -> /AUDIO_IN3
- J3 pad 3: /1POLE_OUT1 -> /1POLE_OUT3
- J3 pad 4: GND -> /FREQ_POT
- J3 pad 5: /AUDIO_IN4 -> GND
- J3 pad 6: GND -> /AUDIO_IN4
- J3 pad 8: /FREQ_JACK -> GND
- J3 pad 9: /1POLE_OUT3 -> /FREQ_CV4
- R28 pad 1: Net-(U1B--) -> Net-(U1D--)
- R29 pad 1: Net-(U1B--) -> Net-(U1D--)
- R30 pad 1: Net-(U1B--) -> Net-(U1D--)
- R31 pad 2: Net-(U1B--) -> Net-(U1D--)
- R56 pad 1: Net-(U1D--) -> Net-(U1B--)
- R57 pad 1: Net-(U1D--) -> Net-(U1B--)
- R58 pad 1: Net-(U1D--) -> Net-(U1B--)
- R59 pad 2: Net-(U1D--) -> Net-(U1B--)
- R65 pad 2: /AUDIO_MIX -> /AUDIO_MIX_1POLE
- R71 pad 2: /AUDIO_MIX -> /AUDIO_MIX_4POLE
- U1 pad 14: /Filter_Voice4/FREQ_CONTROL -> /Filter_Voice2/FREQ_CONTROL
- U1 pad 7: /Filter_Voice2/FREQ_CONTROL -> /Filter_Voice4/FREQ_CONTROL
Routing:
- net /4POLE_OUT4: track 0.00 -> 112.1 mm, vias 0 -> 1
- net /1POLE_OUT3: track 0.00 -> 92.3 mm, vias 0 -> 2
- net /1POLE_OUT4: track 0.00 -> 90.1 mm, vias 0 -> 2
- net /FREQ_JACK: track 0.00 -> 82.1 mm
- net /Q_CONTROL: track 0.00 -> 81.5 mm, vias 0 -> 5
- net /4POLE_OUT3: track 0.00 -> 72.6 mm, vias 0 -> 1
- net /FREQ_POT: track 0.00 -> 66.4 mm, vias 0 -> 1
- net /4POLE_OUT1: track 0.00 -> 56.4 mm
- net /1POLE_OUT2: track 0.00 -> 50.9 mm, vias 0 -> 2
- net /4POLE_OUT2: track 0.00 -> 41.6 mm, vias 0 -> 1
- net /Filter_Voice4/FREQ_CONTROL: track 0.00 -> 39.0 mm
- net /FREQ_CV4: track 0.00 -> 35.3 mm
- net /FREQ_CV3: track 0.00 -> 34.3 mm
- net /1POLE_OUT1: track 0.00 -> 33.6 mm
- net /Filter_Voice1/FREQ_CONTROL: track 0.00 -> 32.1 mm
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
Commit message: Revert "PCB Layout"
This reverts commit f9e64c4088f3b37948fb3949196b7229d7a48ca0.
Parts:
- added Q_POT1: 10k, Custom_Footprints:Alpha_9mm_Potentiometer_Aligned, F.Cu at (135.5, 48.5)
- added kibuzzard-63F9EC4B: G***, kibuzzard-63F9EC4B, F.Cu at (51.6, 119.1)
- added kibuzzard-63F9ECEE: G***, kibuzzard-63F9ECEE, F.Cu at (88.7, 119.1)
- added kibuzzard-63FCE890: G***, kibuzzard-63FCE890, F.Cu at (51.6, 110.9)
- added kibuzzard-63FCEF0D: G***, kibuzzard-63FCEF0D, F.Cu at (88.7, 110.7)
- moved R14 146.8 mm to (194.9, 55.3)
- moved R15 146.8 mm to (194.9, 56.9)
- moved R17 142.1 mm to (194.9, 52.1), turned to 0 degrees
- moved C13 142.1 mm to (194.9, 53.7), turned to 180 degrees
- moved R16 140.9 mm to (194.9, 58.5)
- moved C11 138.0 mm to (205.5, 58.4)
- moved C12 138.0 mm to (205.4, 48.4)
- moved U2 138.0 mm to (205.5, 53.5)
- moved R10 138.0 mm to (211.7, 51.1)
- moved R4 138.0 mm to (199.3, 59.1)
- moved C5 138.0 mm to (199.3, 47.9)
- moved C7 138.0 mm to (199.3, 54.3)
- moved C8 138.0 mm to (199.3, 49.5)
- moved R13 138.0 mm to (199.3, 57.5)
- moved R5 138.0 mm to (199.3, 52.7)
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Connections:
- C22 pad 1: Net-(U1D--) -> Net-(U1B--)
- C40 pad 1: Net-(U1B--) -> Net-(U1D--)
- J1 pad 1: /FREQ_POT_VL -> /FREQ_POT_VH
- J1 pad 10: /FREQ_CV1 -> /AUDIO_IN2
- J1 pad 3: /4POLE_OUT3 -> /4POLE_OUT4
- J1 pad 4: /4POLE_OUT4 -> /FREQ_POT_VL
- J1 pad 5: /AUDIO_MIX_4POLE -> /FREQ_POT
- J1 pad 7: /1POLE_OUT1 -> /FREQ_CV1
- J1 pad 9: /AUDIO_IN1 -> /AUDIO_MIX
- J2 pad 3: /FREQ_POT_VH -> /4POLE_OUT3
- J2 pad 5: /AUDIO_MIX_1POLE -> GND
- J2 pad 8: /AUDIO_IN2 -> /AUDIO_IN1
- J3 pad 1: /FREQ_CV3 -> /AUDIO_IN3
- J3 pad 10: /FREQ_JACK -> /FREQ_CV3
- J3 pad 2: /AUDIO_IN3 -> /FREQ_CV4
- J3 pad 3: /1POLE_OUT3 -> /1POLE_OUT1
- J3 pad 4: /FREQ_POT -> GND
- J3 pad 5: GND -> /AUDIO_IN4
- J3 pad 6: /AUDIO_IN4 -> GND
- J3 pad 8: GND -> /FREQ_JACK
- J3 pad 9: /FREQ_CV4 -> /1POLE_OUT3
- R28 pad 1: Net-(U1D--) -> Net-(U1B--)
- R29 pad 1: Net-(U1D--) -> Net-(U1B--)
- R30 pad 1: Net-(U1D--) -> Net-(U1B--)
- R31 pad 2: Net-(U1D--) -> Net-(U1B--)
- R56 pad 1: Net-(U1B--) -> Net-(U1D--)
- R57 pad 1: Net-(U1B--) -> Net-(U1D--)
- R58 pad 1: Net-(U1B--) -> Net-(U1D--)
- R59 pad 2: Net-(U1B--) -> Net-(U1D--)
- R65 pad 2: /AUDIO_MIX_1POLE -> /AUDIO_MIX
- R71 pad 2: /AUDIO_MIX_4POLE -> /AUDIO_MIX
- U1 pad 14: /Filter_Voice2/FREQ_CONTROL -> /Filter_Voice4/FREQ_CONTROL
- U1 pad 7: /Filter_Voice4/FREQ_CONTROL -> /Filter_Voice2/FREQ_CONTROL
Routing:
- net /4POLE_OUT4: track 112.1 -> 0.00 mm, vias 1 -> 0
- net /1POLE_OUT3: track 92.3 -> 0.00 mm, vias 2 -> 0
- net /1POLE_OUT4: track 90.1 -> 0.00 mm, vias 2 -> 0
- net /FREQ_JACK: track 82.1 -> 0.00 mm
- net /Q_CONTROL: track 81.5 -> 0.00 mm, vias 5 -> 0
- net /4POLE_OUT3: track 72.6 -> 0.00 mm, vias 1 -> 0
- net /FREQ_POT: track 66.4 -> 0.00 mm, vias 1 -> 0
- net /4POLE_OUT1: track 56.4 -> 0.00 mm
- net /1POLE_OUT2: track 50.9 -> 0.00 mm, vias 2 -> 0
- net /4POLE_OUT2: track 41.6 -> 0.00 mm, vias 1 -> 0
- net /Filter_Voice4/FREQ_CONTROL: track 39.0 -> 0.00 mm
- net /FREQ_CV4: track 35.3 -> 0.00 mm
- net /FREQ_CV3: track 34.3 -> 0.00 mm
- net /1POLE_OUT1: track 33.6 -> 0.00 mm
- net /Filter_Voice1/FREQ_CONTROL: track 32.1 -> 0.00 mm
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