File: Hypersoniq.kicad_sch (KiCad schematic)
At the start: 41 parts, among them J1 Conn_01x05_Socket, J2 Conn_01x03_Socket, J3 Conn_01x05_Socket, J4 Conn_01x03_Socket, J5 Conn_01x01_Pin, SW1 ~{LP}_HP, U1 TL072, U2 DG442xY, U4 SSI2140

Commit message: First draft of schematic
Parts:
- removed C10, C11, C8, C9: 1nF, Capacitor_SMD:C_0603_1608Metric_Pad1.08x0.95mm_HandSolder, symbol Device:C_Small
- removed C12, C13, C15, C16: 100nF, Capacitor_SMD:C_0603_1608Metric_Pad1.08x0.95mm_HandSolder, symbol Device:C_Small
- removed C14: 10nF, Capacitor_SMD:C_0603_1608Metric_Pad1.08x0.95mm_HandSolder, symbol Device:C_Small
- removed FREQ_POT1: 10k, Custom_Footprints:Alpha_9mm_Potentiometer_Aligned, symbol Device:R_Potentiometer_Small
- removed J1, J3: Conn_01x05_Socket, Connector_PinSocket_2.54mm:PinSocket_1x05_P2.54mm_Vertical, symbol Connector:Conn_01x05_Socket
- removed J2, J4: Conn_01x03_Socket, Connector_PinSocket_2.54mm:PinSocket_1x03_P2.54mm_Vertical, symbol Connector:Conn_01x03_Socket
- removed J5: Conn_01x01_Pin, Connector_PinHeader_2.54mm:PinHeader_1x01_P2.54mm_Vertical, symbol Connector:Conn_01x01_Pin
- removed R21, R22, R23, R24: 200, Resistor_SMD:R_0603_1608Metric_Pad0.98x0.95mm_HandSolder, symbol Device:R_Small
- removed R25, R26, R27, R28: 10k, Resistor_SMD:R_0603_1608Metric_Pad0.98x0.95mm_HandSolder, symbol Device:R_Small
- removed R29: 1k, Resistor_SMD:R_0603_1608Metric_Pad0.98x0.95mm_HandSolder, symbol Device:R_Small
- removed R30: 54.9, Resistor_SMD:R_0603_1608Metric_Pad0.98x0.95mm_HandSolder, symbol Device:R_Small
- removed R31, R32: 100k, Resistor_SMD:R_0603_1608Metric_Pad0.98x0.95mm_HandSolder, symbol Device:R_Small
- removed R33: 50k, Resistor_SMD:R_0603_1608Metric_Pad0.98x0.95mm_HandSolder, symbol Device:R_Small
- removed R34, R35: 36k, Resistor_SMD:R_0603_1608Metric_Pad0.98x0.95mm_HandSolder, symbol Device:R_Small
- removed R36: 22k, Resistor_SMD:R_0603_1608Metric_Pad0.98x0.95mm_HandSolder, symbol Device:R_Small
- removed R38: 150k, Resistor_SMD:R_0603_1608Metric_Pad0.98x0.95mm_HandSolder, symbol Device:R_Small
- removed SW1: ~{LP}_HP, Custom_Footprints:SPDTSubMiniature, symbol Switch:SW_SPDT
- removed U1: TL072, Package_SO:SO-8_3.9x4.9mm_P1.27mm, symbol Amplifier_Operational:TL072
- removed U2: DG442xY, Package_SO:SOIC-16_3.9x9.9mm_P1.27mm, symbol Analog_Switch:DG442xY
- removed U4: SSI2140, Package_SO:SSOP-20_4.4x6.5mm_P0.65mm, symbol Mountjoy:SSI2140
- added C1, C2: 22uF, Capacitor_SMD:CP_Elec_4x5.8, symbol Device:C_Polarized_Small
- added C41, C42: 100nF, Capacitor_SMD:C_0603_1608Metric_Pad1.08x0.95mm_HandSolder, symbol Device:C_Small
- added D1, D2: 1N5819, Diode_SMD:D_SOD-123, symbol Diode:1N5819
- added J1, J2, J3: Conn_01x10_Pin, Connector_PinHeader_2.54mm:PinHeader_1x10_P2.54mm_Vertical, symbol Connector:Conn_01x10_Pin
- added J4: Eurorack_10_pin_power, Custom_Footprints:Eurorack_10_pin_header, symbol Eurorack_Header:Eurorack_10_pin_power
- added R2: 8.2k, Resistor_SMD:R_0603_1608Metric_Pad0.98x0.95mm_HandSolder, symbol Device:R_Small
- added R3: 3.9k, Resistor_SMD:R_0603_1608Metric_Pad0.98x0.95mm_HandSolder, symbol Device:R_Small
- added R60, R61, R62, R63, R66, R67, R68, R69: 10k, Resistor_SMD:R_0603_1608Metric_Pad0.98x0.95mm_HandSolder, symbol Device:R_Small
- added R64, R70: 4.7k, Resistor_SMD:R_0603_1608Metric_Pad0.98x0.95mm_HandSolder, symbol Device:R_Small
- added R65, R71: 1k, Resistor_SMD:R_0603_1608Metric_Pad0.98x0.95mm_HandSolder, symbol Device:R_Small
- added TP2, TP3, TP4: TestPoint, Custom_Footprints:1.3mm_Test_Point, symbol Connector:TestPoint
- added U1: TL074, Package_SO:SOIC-14_3.9x8.7mm_P1.27mm, symbol Amplifier_Operational:TL074
- added U6: TL072, Package_SO:SO-8_3.9x4.9mm_P1.27mm, symbol Amplifier_Operational:TL072
- R1: renamed from R37; value 22k -> 39k
- TP1: now left out of the parts list
- renumbered C18 to C3, C17 to C4
Connections:
- net +12V: now also TP1.1, C1.1, C41.1, D1.1 (K), J2.1 (Pin_1), R2.1, U1.4 (V+), U6.4 (V-)
- net -12V: now also C2.2, C42.1, D2.2 (A), R3.2, TP2.1, U1.11 (V-), U6.8 (V+)
- net FREQ_CV1: now also J1.7 (Pin_7)
- net FREQ_CV2: now also J2.10 (Pin_10)
- net FREQ_POT: now also J1.5 (Pin_5)
- net GND: now also C1.2, C2.1, C41.2, C42.2, J1.6 (Pin_6), J2.5 (Pin_5), J2.6 (Pin_6), J2.7 (Pin_7), J3.4 (Pin_4), J3.6 (Pin_6), J3.7 (Pin_7), J4.3 (Pin_3), J4.4 (Pin_4), J4.5 (Pin_5), J4.6 (Pin_6), J4.7 (Pin_7), J4.8 (Pin_8), TP3.1, TP4.1, U6.3 (+), U6.5 (+); no longer TP1.1
- net Q_POT: now reaches Q_POT1.2, R1.1
- net Q_POT: now also J1.8 (Pin_8)
- new net: R60.1, R61.1, R62.1, R63.1, R64.2, U6.2 (-)
- new net: R66.1, R67.1, R68.1, R69.1, R70.2, U6.6 (-)
- new net: R70.1, R71.1, U6.7
- new net: R64.1, R65.1, U6.1
- new net +12V_IN: D1.2 (A), J4.10 (Pin_10), J4.9 (Pin_9)
- new net -12V_IN: D2.1 (K), J4.1 (Pin_1), J4.2 (Pin_2)
- new net 1POLE_OUT1: J3.3 (Pin_3), R60.2
- new net 1POLE_OUT2: J2.9 (Pin_9), R61.2
- new net 1POLE_OUT3: J3.9 (Pin_9), R62.2
- new net 1POLE_OUT4: J2.4 (Pin_4), R63.2
- new net 4POLE_OUT1: J2.2 (Pin_2), R66.2
- new net 4POLE_OUT2: J1.2 (Pin_2), R67.2
- new net 4POLE_OUT3: J2.3 (Pin_3), R68.2
- new net 4POLE_OUT4: J1.3 (Pin_3), R69.2
- new net AUDIO_IN1: J2.8 (Pin_8)
- new net AUDIO_IN2: J1.10 (Pin_10)
- new net AUDIO_IN3: J3.1 (Pin_1)
- new net AUDIO_IN4: J3.5 (Pin_5)
- new net AUDIO_MIX: J1.9 (Pin_9), R65.2, R71.2
- new net FREQ_CV3: J3.10 (Pin_10)
- new net FREQ_CV4: J3.2 (Pin_2)
- new net FREQ_JACK: J3.8 (Pin_8)
- new net FREQ_POT_VH: J1.1 (Pin_1), R2.2
- new net FREQ_POT_VL: J1.4 (Pin_4), R3.1
Other:
- added sheet Filter_Voice1 (Filter_Voice.kicad_sch)
- added sheet Filter_Voice2 (Filter_Voice.kicad_sch)
- added sheet Filter_Voice3 (Filter_Voice.kicad_sch)
- added sheet Filter_Voice4 (Filter_Voice.kicad_sch)
- note added: "Gain: -4.7k / 10k = -0.47"
- note added: "HP Filter Voices"
- note added: "Interconnects and Test Points"
- note added: "Measured Pot Range: -7.5v to 2.75v"
- note added: "Q Control: Ground-referenced current input"
- note removed: "12v x 10k / (10k + 36k) = 2.61V"
- note removed: "HP Filter"
- note removed: "Mixed Mode HP/LP"
- note removed: "Q Control: Ground-referenced current input Input Current Range 0-500uA 22k resistor means an input voltage of 11v gives 500uA"
- note removed: "v2 Fix: HP Only design connnect Q_VCA_OUT to pin 6"
- moved on the sheet: C3, C4, Q_POT1, R1

Commit message: Revert "Revert "PCB Layout""
This reverts commit 17ea893c43406ccb0184a474adf0eed468bf1595.
Parts:
- removed Q_POT1: 10k, Custom_Footprints:Alpha_9mm_Potentiometer_Aligned, symbol Device:R_Potentiometer_Small
Connections:
- net 1POLE_OUT1: now also J1.7 (Pin_7); no longer J3.3 (Pin_3)
- net 1POLE_OUT3: now also J3.3 (Pin_3); no longer J3.9 (Pin_9)
- net 4POLE_OUT3: now also J1.3 (Pin_3); no longer J2.3 (Pin_3)
- net 4POLE_OUT4: now also J1.4 (Pin_4); no longer J1.3 (Pin_3)
- net AUDIO_IN1: now also J1.9 (Pin_9); no longer J2.8 (Pin_8)
- net AUDIO_IN2: now also J2.8 (Pin_8); no longer J1.10 (Pin_10)
- net AUDIO_IN3: now also J3.2 (Pin_2); no longer J3.1 (Pin_1)
- net AUDIO_IN4: now also J3.6 (Pin_6); no longer J3.5 (Pin_5)
- net FREQ_CV1: now also J1.10 (Pin_10); no longer J1.7 (Pin_7)
- net FREQ_CV3: now also J3.1 (Pin_1); no longer J3.10 (Pin_10)
- net FREQ_CV4: now also J3.9 (Pin_9); no longer J3.2 (Pin_2)
- net FREQ_JACK: now also J3.10 (Pin_10); no longer J3.8 (Pin_8)
- net FREQ_POT: now also J3.4 (Pin_4); no longer J1.5 (Pin_5)
- net FREQ_POT_VH: now also J2.3 (Pin_3); no longer J1.1 (Pin_1)
- net FREQ_POT_VL: now also J1.1 (Pin_1); no longer J1.4 (Pin_4)
- net GND: now also J3.5 (Pin_5), J3.8 (Pin_8); no longer J2.5 (Pin_5), J3.4 (Pin_4), J3.6 (Pin_6)
- removed net AUDIO_MIX: J1.9 (Pin_9), R65.2, R71.2
- new net AUDIO_MIX_1POLE: J2.5 (Pin_5), R65.2
- new net AUDIO_MIX_4POLE: J1.5 (Pin_5), R71.2
Other:
- note added: "Q Pot: 10k between +12V and GND Q Control: Ground-referenced current input"
- note removed: "Q Control: Ground-referenced current input"

Commit message: Revert "PCB Layout"
This reverts commit f9e64c4088f3b37948fb3949196b7229d7a48ca0.
Parts:
- added Q_POT1: 10k, Custom_Footprints:Alpha_9mm_Potentiometer_Aligned, symbol Device:R_Potentiometer_Small
Connections:
- net +12V: now also Q_POT1.1
- net 1POLE_OUT1: now also J3.3 (Pin_3); no longer J1.7 (Pin_7)
- net 1POLE_OUT3: now also J3.9 (Pin_9); no longer J3.3 (Pin_3)
- net 4POLE_OUT3: now also J2.3 (Pin_3); no longer J1.3 (Pin_3)
- net 4POLE_OUT4: now also J1.3 (Pin_3); no longer J1.4 (Pin_4)
- net AUDIO_IN1: now also J2.8 (Pin_8); no longer J1.9 (Pin_9)
- net AUDIO_IN2: now also J1.10 (Pin_10); no longer J2.8 (Pin_8)
- net AUDIO_IN3: now also J3.1 (Pin_1); no longer J3.2 (Pin_2)
- net AUDIO_IN4: now also J3.5 (Pin_5); no longer J3.6 (Pin_6)
- net FREQ_CV1: now also J1.7 (Pin_7); no longer J1.10 (Pin_10)
- net FREQ_CV3: now also J3.10 (Pin_10); no longer J3.1 (Pin_1)
- net FREQ_CV4: now also J3.2 (Pin_2); no longer J3.9 (Pin_9)
- net FREQ_JACK: now also J3.8 (Pin_8); no longer J3.10 (Pin_10)
- net FREQ_POT: now also J1.5 (Pin_5); no longer J3.4 (Pin_4)
- net FREQ_POT_VH: now also J1.1 (Pin_1); no longer J2.3 (Pin_3)
- net FREQ_POT_VL: now also J1.4 (Pin_4); no longer J1.1 (Pin_1)
- net GND: now also J2.5 (Pin_5), J3.4 (Pin_4), J3.6 (Pin_6), Q_POT1.3; no longer J3.5 (Pin_5), J3.8 (Pin_8)
- net Q_POT: now also Q_POT1.2
- net AUDIO_MIX_1POLE renamed AUDIO_MIX
- net AUDIO_MIX: now also J1.9 (Pin_9), R71.2; no longer J2.5 (Pin_5)
- removed net AUDIO_MIX_4POLE: J1.5 (Pin_5), R71.2
Other:
- note added: "Q Control: Ground-referenced current input"
- note removed: "Q Pot: 10k between +12V and GND Q Control: Ground-referenced current input"
