File: Hypersoniq_Controls.kicad_sch (KiCad schematic)
At the start: 15 parts, among them J1 Conn_01x10_Pin, J11 Freq_In, J12 Audio_Mix_4Pole, J2 Conn_01x10_Pin, J3 Conn_01x10_Pin, J4 Audio_In, J5 Audio_Out_1P, J6 Audio_Mix_1Pole, J7 Freq_CV, J8 Audio_Out_4P

Commit message: v1.0 Design sent for manufacture
Parts:
- J1, J2, J3: footprint Connector_PinHeader_2.54mm:PinHeader_1x10_P2.54mm_Vertical -> Connector_PinSocket_2.54mm:PinSocket_1x10_P2.54mm_Vertical; symbol Connector:Conn_01x10_Pin -> Connector:Conn_01x10_Socket
Connections:
- net GND: no longer J3.5 (Pin_5)
- new net -12V: J3.5 (Pin_5)
